File: pcm_pmod.kicad_sch (KiCad schematic)
At the start: 12 parts, among them J1 pmod, J2 +5V, J3 AudioJack4, U1 pcm_adc, U2 inmp441, U3 inmp441

Commit message: add screenshots
Other:
- company: (none) -> S59MZ
